File: Group_06/Group_06.brd (EAGLE design)
At the start: 72.4 x 60.8 mm, 29 parts, among them J1 POWER_JACKPTH_LOCK, U2 +12v

Commit message: update board
Parts:
- moved C1 2.54 mm to (47.0, 11.2)
- moved C2 1.53 mm to (46.9, 3.43)
Changed lines of the file:
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@@
 <drawing>
 <settings>
-<setting alwaysvectorfont="yes"/>
+<setting alwaysvectorfont="no"/>
 <setting verticaltext="up"/>
 </settings>
@@
 <text x="13.843" y="28.448" size="1.6764" layer="21" font="vector" ratio="15">DEVELOPMENT</text>
 <text x="13.843" y="25.908" size="1.6764" layer="21" font="vector" ratio="15">KIT PSOC-5LP</text>
-<text x="11.43" y="7.747" size="0.6096" layer="21" font="vector" ratio="15">LIGHT SENSOR</text>
+<text x="11.811" y="7.747" size="0.6096" layer="21" font="vector" ratio="15">LIGHT SENSOR</text>
 <text x="22.098" y="11.811" size="0.6096" layer="21" font="vector" ratio="15">TEMPERATURE
 SENSOR</text>
@@
 <text x="29.972" y="10.414" size="0.6096" layer="21" font="vector" ratio="15">5V</text>
 <text x="33.274" y="15.875" size="0.6096" layer="21" font="vector" ratio="15">V. REG</text>
-<text x="47.625" y="5.207" size="0.508" layer="21" font="vector" ratio="15">0.1 uF</text>
+<text x="46.101" y="5.207" size="0.508" layer="21" font="vector" ratio="15">0.1 uF</text>
 <text x="24.13" y="48.514" size="0.508" layer="21" font="vector" ratio="15">0.1 uF</text>
-<text x="16.383" y="4.953" size="0.6096" layer="21" font="vector" ratio="15">330</text>
-<text x="48.006" y="10.033" size="0.508" layer="21" font="vector" ratio="15" rot="R90">0.33 uF</text>
-<text x="8.255" y="10.16" size="0.508" layer="21" font="vector" ratio="15" rot="R90">10K</text>
+<text x="16.002" y="3.556" size="0.6096" layer="21" font="vector" ratio="15">330</text>
+<text x="45.466" y="10.033" size="0.508" layer="21" font="vector" ratio="15" rot="R90">0.33 uF</text>
+<text x="9.906" y="10.414" size="0.508" layer="21" font="vector" ratio="15" rot="R90">10K</text>
 <text x="2.286" y="9.017" size="0.6096" layer="21" font="vector" ratio="15" rot="R90">BLUE LED</text>
 <text x="25.019" y="44.45" size="0.6096" layer="25" font="vector" ratio="15">C3</text>
-<text x="48.006" y="1.27" size="0.6096" layer="25" font="vector" ratio="15">C2</text>
+<text x="46.482" y="1.27" size="0.6096" layer="25" font="vector" ratio="15">C2</text>
 <text x="49.276" y="55.372" size="0.4064" layer="21" font="vector" ratio="15">8x 4.7K</text>
 <circle x="69.85" y="2.54" radius="1.849146875" width="0.254" layer="21"/>
@@
 <wire x1="7.747" y1="9.144" x2="9.017" y2="9.144" width="0.1016" layer="21"/>
 <wire x1="4.318" y1="10.668" x2="5.08" y2="10.668" width="0.1016" layer="21"/>
-<wire x1="48.768" y1="12.827" x2="50.292" y2="12.827" width="0.1016" layer="21"/>
-<wire x1="48.895" y1="9.525" x2="50.165" y2="9.525" width="0.1016" layer="21"/>
+<wire x1="46.228" y1="12.827" x2="47.752" y2="12.827" width="0.1016" layer="21"/>
+<wire x1="46.355" y1="9.525" x2="47.625" y2="9.525" width="0.1016" layer="21"/>
 <wire x1="4.191" y1="11.176" x2="5.207" y2="11.176" width="0.1016" layer="21"/>
 <dimension x1="0" y1="60.833" x2="72.39" y2="60.833" x3="36.195" y3="66.04" textsize="1.778" layer="20"/>
@@
 <param name="dpMaxLengthDifference" value="10mm"/>
 <param name="dpGapFactor" value="2.5"/>
-<param name="checkAngle" value="0"/>
+<param name="checkAngle" value="1"/>
 <param name="checkFont" value="1"/>
 <param name="checkRestrict" value="1"/>
 <param name="checkStop" value="0"/>
-<param name="checkValues" value="0"/>
+<param name="checkValues" value="1"/>
 <param name="checkNames" value="1"/>
 <param name="checkWireStubs" value="1"/>
@@
 </element>
 <element name="R1" library="SparkFun-Sensors" package="PHOTOCELL" value="PHOTOCELLPTH" x="14.478" y="11.303" smashed="yes">
-<attribute name="NAME" x="13.589" y="14.351" size="0.6096" layer="25" font="vector" ratio="20" rot="R180" align="bottom-center"/>
+<attribute name="NAME" x="14.478" y="14.224" size="0.6096" layer="25" font="vector" ratio="20" rot="R180" align="bottom-center"/>
 <attribute name="PROD_ID" value="COMP-09129" x="14.478" y="11.303" size="1.778" layer="27" font="vector" ratio="15" display="off"/>
 <attribute name="SF_ID" value="SEN-09088" x="14.478" y="11.303" size="1.778" layer="27" font="vector" ratio="15" display="off"/>
@@
 <attribute name="VALUE" x="73.025" y="7.747" size="0.6096" layer="27" font="vector" ratio="20" rot="R90"/>
 </element>
-<element name="C1" library="SparkFun-Capacitors" package="0805" value="0.33µF" x="49.53" y="11.176" smashed="yes" rot="R270">
-<attribute name="NAME" x="50.8" y="11.176" size="0.6096" layer="25" font="vector" ratio="20" rot="R270" align="bottom-center"/>
-<attribute name="PROD_ID" value="CAP-08469" x="49.53" y="11.176" size="1.778" layer="27" font="vector" ratio="15" rot="R270" display="off"/>
-<attribute name="VALUE" x="48.641" y="11.176" size="0.6096" layer="27" font="vector" ratio="20" rot="R270" align="top-center"/>
-</element>
-<element name="C2" library="SparkFun-Capacitors" package="CAP-PTH-SMALL-KIT" value="0.1uF" x="48.387" y="3.556" smashed="yes" rot="R180">
-<attribute name="PROD_ID" value="CAP-08370" x="48.387" y="3.556" size="1.778" layer="27" font="vector" ratio="15" rot="R180" display="off"/>
+<element name="C1" library="SparkFun-Capacitors" package="0805" value="0.33µF" x="46.99" y="11.176" smashed="yes" rot="R270">
+<attribute name="NAME" x="48.26" y="11.176" size="0.6096" layer="25" font="vector" ratio="20" rot="R270" align="bottom-center"/>
+<attribute name="PROD_ID" value="CAP-08469" x="46.99" y="11.176" size="1.778" layer="27" font="vector" ratio="15" rot="R270" display="off"/>
+<attribute name="VALUE" x="46.101" y="11.176" size="0.6096" layer="27" font="vector" ratio="20" rot="R270" align="top-center"/>
+</element>
+<element name="C2" library="SparkFun-Capacitors" package="CAP-PTH-SMALL-KIT" value="0.1uF" x="46.863" y="3.429" smashed="yes" rot="R180">
+<attribute name="PROD_ID" value="CAP-08370" x="46.863" y="3.429" size="1.778" layer="27" font="vector" ratio="15" rot="R180" display="off"/>
 </element>
 <element name="U2" library="SparkFun-IC-Power" package="TO-252" value="+12v" x="35.179" y="11.557" smashed="yes" rot="R270">
@@
 </element>
 <element name="J7" library="SparkFun-Connectors" package="1X02" value="" x="35.56" y="57.658" smashed="yes">
-<attribute name="NAME" x="36.322" y="59.436" size="0.6096" layer="25" font="vector" ratio="20"/>
+<attribute name="NAME" x="36.449" y="59.563" size="0.6096" layer="25" font="vector" ratio="20"/>
 <attribute name="VALUE" x="34.29" y="55.626" size="0.6096" layer="27" font="vector" ratio="20"/>
 </element>
@@
 <element name="U$2" library="CY8KIT-059" package="CY8CKIT-059_TARGET" value="CY8CKIT-059_TARGET" x="37.846" y="30.861" smashed="yes"/>
 <element name="J8" library="SparkFun-Connectors" package="1X08_LOCK" value="" x="6.477" y="57.658" smashed="yes">
-<attribute name="NAME" x="5.207" y="59.055" size="0.6096" layer="25" font="vector" ratio="20"/>
+<attribute name="NAME" x="14.859" y="59.436" size="0.6096" layer="25" font="vector" ratio="20"/>
 <attribute name="VALUE" x="5.207" y="55.626" size="0.6096" layer="27" font="vector" ratio="20"/>
 </element>
@@
 <wire x1="54.864" y1="17.653" x2="52.324" y2="15.113" width="0.254" layer="16"/>
 <wire x1="52.324" y1="15.113" x2="52.324" y2="3.429" width="0.254" layer="16"/>
-<wire x1="52.324" y1="3.429" x2="49.911" y2="3.429" width="0.254" layer="16"/>
-<wire x1="49.911" y1="3.429" x2="49.784" y2="3.556" width="0.254" layer="16"/>
+<wire x1="52.324" y1="3.429" x2="48.26" y2="3.429" width="0.254" layer="16"/>
 <wire x1="16.694" y1="50.003" x2="17.11" y2="50.003" width="0.2032" layer="1"/>
 <wire x1="17.272" y1="50.165" x2="17.653" y2="50.165" width="0.2032" layer="1"/>
@@
 <wire x1="26.67" y1="46.863" x2="26.67" y2="50.038" width="0.2032" layer="1"/>
 <wire x1="26.67" y1="50.038" x2="23.368" y2="53.34" width="0.2032" layer="1"/>
-<wire x1="49.784" y1="3.556" x2="49.53" y2="3.81" width="0.254" layer="1"/>
-<wire x1="49.53" y1="3.81" x2="49.53" y2="6.35" width="0.254" layer="1"/>
-<wire x1="49.53" y1="6.35" x2="48.26" y2="7.62" width="0.254" layer="1"/>
-<wire x1="48.26" y1="7.62" x2="30.48" y2="7.62" width="0.254" layer="1"/>
+<wire x1="48.26" y1="6.477" x2="48.26" y2="3.429" width="0.254" layer="1"/>
+<wire x1="48.26" y1="6.477" x2="47.117" y2="7.62" width="0.254" layer="1"/>
+<wire x1="47.117" y1="7.62" x2="30.48" y2="7.62" width="0.254" layer="1"/>
 <wire x1="28.468" y1="7.366" x2="24.638" y2="7.366" width="0.254" layer="1"/>
 <wire x1="30.48" y1="7.62" x2="30.379" y2="7.721" width="0.254" layer="1"/>
@@
 <contactref element="S1" pad="1"/>
 <wire x1="30.363" y1="13.853" x2="30.379" y2="13.837" width="0.254" layer="1"/>
-<wire x1="55.499" y1="12.192" x2="49.646" y2="12.192" width="0.254" layer="1"/>
-<wire x1="49.646" y1="12.192" x2="49.53" y2="12.076" width="0.254" layer="1"/>
-<wire x1="49.53" y1="12.076" x2="49.53" y2="15.24" width="0.254" layer="1"/>
-<wire x1="48.895" y1="15.875" x2="30.363" y2="15.875" width="0.254" layer="1"/>
-<wire x1="49.53" y1="15.24" x2="48.895" y2="15.875" width="0.254" layer="1"/>
+<wire x1="55.499" y1="12.192" x2="47.106" y2="12.192" width="0.254" layer="1"/>
+<wire x1="47.106" y1="12.192" x2="46.99" y2="12.076" width="0.254" layer="1"/>
+<wire x1="46.99" y1="12.076" x2="46.99" y2="15.875" width="0.254" layer="1"/>
+<wire x1="46.99" y1="15.875" x2="30.363" y2="15.875" width="0.254" layer="1"/>
 <wire x1="30.363" y1="15.875" x2="30.363" y2="13.853" width="0.254" layer="1"/>
 </signal>
